File: schematic.brd (EAGLE design)
At the start: 20.3 x 127 mm, 13 parts

Commit message: Updates
Parts:
- added C1, C2: (no value), rcl:E2,5-4R
- added R2, R3: 1K, rcl:0204/5
- moved PWR 3.41 mm to (7.11, 3.56)
- moved D1 0.51 mm to (18.2, 23.3)
- moved OPAMP1 0.51 mm to (5.54, 24.1)
- moved OPAMP2 0.51 mm to (5.49, 14.4)
- moved R1 0.51 mm to (18.3, 12.7)
Connections:
- new net N$11: C1.+, R3.1
- new net N$12: C2.-, R2.2
- net +12V: now also C2.+, R2.1
- net -12V: now also C1.-, R3.2
Routing:
- net N$5: track 45.7 -> 23.3 mm
- net N$7: track 19.0 -> 37.7 mm
- net +5V: track 113.5 -> 127.1 mm
- net -12V: track 19.0 -> 32.0 mm
- net N$6: track 87.5 -> 75.2 mm
- net N$3: track 33.0 -> 25.1 mm
- net N$12: track 0.00 -> 7.82 mm
- net N$11: track 0.00 -> 6.55 mm
- net N$4: track 79.3 -> 73.7 mm
- net +12V: track 45.6 -> 49.5 mm
- net GND: track 160.9 -> 157.6 mm
- net N$8: track 43.3 -> 44.5 mm
- net N$1: track 100.2 -> 99.7 mm

Commit message: Updates
Parts:
- moved R1 7.33 mm to (14.2, 18.8)
- moved R3 7.33 mm to (18.3, 12.7)
Connections:
- net +12V: now also R3.2; no longer R1.2
- net +5V: now also R3.1; no longer R1.1
- net -12V: now also R1.2; no longer R3.2
- net N$11: now also R1.1; no longer R3.1
Changed lines of the file:
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@@
 <attribute name="NAME" x="0.5588" y="55.5244" size="1.016" layer="21" rot="SR0"/>
 </element>
-<element name="R1" library="rcl" library_urn="urn:adsk.eagle:library:334" package="0204/5" package3d_urn="urn:adsk.eagle:package:23488/1" value="1K" x="18.288" y="12.7" smashed="yes" rot="R270">
+<element name="R3" library="rcl" library_urn="urn:adsk.eagle:library:334" package="0204/5" package3d_urn="urn:adsk.eagle:package:23488/1" value="1K" x="18.288" y="12.7" smashed="yes" rot="R270">
 <attribute name="MF" value="VISHAY" x="18.288" y="12.7" size="1.778" layer="27" rot="R270" display="off"/>
 <attribute name="MPN" value="CCF551K00FKE36" x="18.288" y="12.7" size="1.778" layer="27" rot="R270" display="off"/>
@@
 <attribute name="VALUE" x="11.9126" y="12.8016" size="0.9906" layer="27" ratio="10" rot="R270"/>
 </element>
-<element name="R3" library="rcl" library_urn="urn:adsk.eagle:library:334" package="0204/5" package3d_urn="urn:adsk.eagle:package:23488/1" value="1K" x="14.224" y="18.796" smashed="yes" rot="R270">
+<element name="R1" library="rcl" library_urn="urn:adsk.eagle:library:334" package="0204/5" package3d_urn="urn:adsk.eagle:package:23488/1" value="1K" x="14.224" y="18.796" smashed="yes" rot="R270">
 <attribute name="MF" value="VISHAY" x="14.224" y="18.796" size="1.778" layer="27" rot="R270" display="off"/>
 <attribute name="MPN" value="CCF551K00FKE36" x="14.224" y="18.796" size="1.778" layer="27" rot="R270" display="off"/>
@@
 <signals>
 <signal name="+12V">
-<contactref element="R1" pad="2"/>
+<contactref element="R3" pad="2"/>
 <contactref element="PWR" pad="10"/>
 <contactref element="PWR" pad="9"/>
@@
 <signal name="+5V">
 <contactref element="VR1" pad="1"/>
-<contactref element="R1" pad="1"/>
+<contactref element="R3" pad="1"/>
 <contactref element="D1" pad="1"/>
 <contactref element="VR2" pad="1"/>
@@
 <contactref element="OPAMP1" pad="4"/>
 <contactref element="C1" pad="-"/>
-<contactref element="R3" pad="2"/>
+<contactref element="R1" pad="2"/>
 <wire x1="1.9558" y1="4.7498" x2="1.9558" y2="2.5146" width="0.3048" layer="1"/>
 <wire x1="1.9558" y1="2.5146" x2="2.032" y2="2.286" width="0.3048" layer="1"/>
@@
 <signal name="N$11">
 <contactref element="C1" pad="+"/>
-<contactref element="R3" pad="1"/>
+<contactref element="R1" pad="1"/>
 <wire x1="13.97" y1="22.6314" x2="13.97" y2="21.5138" width="0.3048" layer="16"/>
 <wire x1="12.8524" y1="23.749" x2="13.97" y2="22.6314" width="0.3048" layer="16"/>
