File: schematic.sch (EAGLE design)
At the start: 17 parts

Commit message: Updates
Connections:
- net +12V: now also R3.2; no longer R1.2
- net +5V: now also R3.1; no longer R1.1
- net -12V: now also R1.2; no longer R3.2
- net N$11: now also R1.1; no longer R3.1
Other:
- moved on the sheet: R1, R3
Changed lines of the file:
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@@
 </modules>
 <parts>
-<part name="R1" library="rcl" library_urn="urn:adsk.eagle:library:334" deviceset="R-EU_" device="0204/5" package3d_urn="urn:adsk.eagle:package:23488/1" value="1K">
+<part name="R3" library="rcl" library_urn="urn:adsk.eagle:library:334" deviceset="R-EU_" device="0204/5" package3d_urn="urn:adsk.eagle:package:23488/1" value="1K">
 <spice>
 <pinmapping spiceprefix="R">
@@
 <attribute name="OC_NEWARK" value="71M1025"/>
 </part>
-<part name="R3" library="rcl" library_urn="urn:adsk.eagle:library:334" deviceset="R-EU_" device="0204/5" package3d_urn="urn:adsk.eagle:package:23488/1" value="1K">
+<part name="R1" library="rcl" library_urn="urn:adsk.eagle:library:334" deviceset="R-EU_" device="0204/5" package3d_urn="urn:adsk.eagle:package:23488/1" value="1K">
 <spice>
 <pinmapping spiceprefix="R">
@@
 </plain>
 <instances>
-<instance part="R1" gate="G$1" x="-7.62" y="76.2" smashed="yes" rot="R90">
+<instance part="R3" gate="G$1" x="-7.62" y="76.2" smashed="yes" rot="R90">
 <attribute name="NAME" x="-9.1186" y="72.39" size="1.778" layer="95" rot="R90"/>
 <attribute name="VALUE" x="-4.318" y="72.39" size="1.778" layer="96" rot="R90"/>
@@
 <attribute name="MPN" x="-30.48" y="83.82" size="1.778" layer="96" display="off"/>
 </instance>
-<instance part="R3" gate="G$1" x="-30.48" y="53.34" smashed="yes" rot="R90">
+<instance part="R1" gate="G$1" x="-30.48" y="53.34" smashed="yes" rot="R90">
 <attribute name="NAME" x="-31.9786" y="49.53" size="1.778" layer="95" rot="R90"/>
 <attribute name="VALUE" x="-27.178" y="49.53" size="1.778" layer="96" rot="R90"/>
@@
 <segment>
 <pinref part="P+1" gate="1" pin="+12V"/>
-<pinref part="R1" gate="G$1" pin="2"/>
+<pinref part="R3" gate="G$1" pin="2"/>
 <wire x1="-7.62" y1="86.36" x2="-7.62" y2="81.28" width="0.1524" layer="91"/>
 </segment>
@@
 </segment>
 <segment>
-<pinref part="R1" gate="G$1" pin="1"/>
+<pinref part="R3" gate="G$1" pin="1"/>
 <pinref part="D1" gate="G$0" pin="CATHODE"/>
 <wire x1="-7.62" y1="71.12" x2="-7.62" y2="66.04" width="0.1524" layer="91"/>
@@
 <wire x1="-40.64" y1="66.04" x2="-38.1" y2="66.04" width="0.1524" layer="91"/>
 <wire x1="-38.1" y1="66.04" x2="-38.1" y2="58.42" width="0.1524" layer="91"/>
-<pinref part="R3" gate="G$1" pin="2"/>
+<pinref part="R1" gate="G$1" pin="2"/>
 <wire x1="-38.1" y1="58.42" x2="-30.48" y2="58.42" width="0.1524" layer="91"/>
 <junction x="-38.1" y="58.42"/>
@@
 <pinref part="C1" gate="G$1" pin="+"/>
 <wire x1="-38.1" y1="50.8" x2="-38.1" y2="48.26" width="0.1524" layer="91"/>
-<pinref part="R3" gate="G$1" pin="1"/>
+<pinref part="R1" gate="G$1" pin="1"/>
 <wire x1="-38.1" y1="48.26" x2="-30.48" y2="48.26" width="0.1524" layer="91"/>
 <wire x1="-30.48" y1="48.26" x2="-30.48" y2="43.18" width="0.1524" layer="91"/>
